Commit message: Fixing robot sdf bug, creating new sdf for sorting shelf

File: manipulation/models/iiwa_description/urdf/iiwa7_no_world_joint.urdf (robot description, URDF)
Before this commit: robot iiwa7, 10 links, 9 joints
Links:
- removed link iiwa_link_7
- removed link iiwa_link_ee
- removed link iiwa_link_ee_kuka
- link iiwa_link_1: mass 4 -> None
- link iiwa_link_2: mass 4 -> None
- link iiwa_link_3: mass 3 -> None
- link iiwa_link_4: mass 2.7 -> None
- link iiwa_link_5: mass 1.7 -> None
- link iiwa_link_6: mass 1.8 -> None
Joints:
- removed joint iiwa_joint_7
- removed joint iiwa_joint_ee
- removed joint tool0_joint

File: manipulation/models/yaskawa_description/urdf/yaskawa_no_collision.urdf (robot description, URDF)
Before this commit: robot yaskawa, 10 links, 9 joints
Links:
- removed link ee_mount
- link b_link: mass 2.7 -> None; geometry visual mesh filename=../mesh/b-visual2.obj scale=1 1 1
- link f_link: mass 4 -> None
- link l_link: mass 4 -> None
- link r_link: mass 1.7 -> None
- link s_link: mass 4 -> None
- link t_link: geometry visual mesh filename=../mesh/t-visual.obj scale=1 1 1
- link u_link: mass 4 -> None
Joints:
- removed joint ee_mount_joint
- joint b_joint: axis 0 0 1 -> 0 -1 0
- joint f_joint: origin xyz=0.0 0.0 0.8 rpy=0 0 0 -> xyz=0.0 0.0 0.71 rpy=0 0 0
- joint r_joint: axis 0 0 1 -> -1 0 0; origin xyz=0.295 0.066 0.200 rpy=0 0 1.75 -> xyz=0.295 0.066 0.200 rpy=0 0 0
- joint t_joint: axis 0 0 1 -> -1 0 0
- joint u_joint: axis 0 0 1 -> 0 -1 0
