Commit message: Put in robot arm base and 1 cabinet

File: manipulation/models/yaskawa_description/urdf/yaskawa_no_collision.urdf (robot description, URDF)
Before this commit: robot yaskawa, 9 links, 8 joints
Links:
- added link gp25_fixed_base_link; visual mesh filename=../mesh/gp25_base_700.obj
Joints:
- added joint mh25_fixed_base_link_joint: type fixed, parent arm_base, child gp25_fixed_base_link, origin xyz=0 0 0 rpy=0 0 0
- joint f_joint: origin xyz=0.0 0.0 0.0 rpy=0 0 0 -> xyz=0.0 0.0 0.7 rpy=0 0 0; parent arm_base -> gp25_fixed_base_link

Commit message: Added 2 more sorting shelves and currently fixing robot bug. Solution is to define correct inertia parameters in the URDF file

File: manipulation/models/yaskawa_description/urdf/yaskawa_no_collision.urdf (robot description, URDF)
Before this commit: robot yaskawa, 10 links, 9 joints
Links:
- link arm_base: geometry 
- link b_link: mass None -> 2.7
- link ee_mount: geometry 
- link f_link: mass None -> 4
- link l_link: mass None -> 4
- link r_link: mass None -> 1.7
- link s_link: mass None -> 4
- link t_link: geometry 
- link u_link: mass None -> 4
Joints:
- joint b_joint: axis 0 -1 0 -> 0 0 1
- joint f_joint: origin xyz=0.0 0.0 0.7 rpy=0 0 0 -> xyz=0.0 0.0 0.8 rpy=0 0 0
- joint r_joint: axis -1 0 0 -> 0 0 1; origin xyz=0.295 0.066 0.200 rpy=0 0 0 -> xyz=0.295 0.066 0.200 rpy=0 0 1.75
- joint t_joint: axis -1 0 0 -> 0 0 1
- joint u_joint: axis 0 -1 0 -> 0 0 1

Commit message: Created conveyor belt and put in packages. Working on getting the gripper model to the correct size

File: manipulation/models/yaskawa_description/urdf/yaskawa_no_collision.urdf (robot description, URDF)
Before this commit: robot yaskawa, 9 links, 8 joints
Links:
- added link ee_mount
- link b_link: mass None -> 2.4338
- link f_link: mass None -> 9.3324
- link l_link: mass None -> 5.7076
- link r_link: mass None -> 4.0138
- link s_link: mass None -> 15.959
- link t_link: mass None -> 0.61827
- link u_link: mass None -> 7.4543
Joints:
- added joint ee_mount_joint: type fixed, parent t_link, child ee_mount, origin xyz=0.0 0.0 0.0 rpy=0 0 0
