Commit message: Put in new ee for yaskawa. Problem: Failure at multibody/plant/tamsi_solver.cc:217 in SolveQuadraticForTheSmallestPositiveRoot(): condition 'Delta > 0' failed

File: manipulation/models/allegro_hand_description/urdf/allegro_hand_description_right.urdf (robot description, URDF)
Before this commit: robot allegro_hand_right, 22 links, 21 joints
Links:
- removed link hand_root
- added link ee_base
Joints:
- joint root_to_base: parent hand_root -> ee_base
