Commit message: fixing end effector. Creating new controller for it

File: manipulation/models/yaskawa_end_effector_description/urdf/end_effector_3.urdf (robot description, URDF)
Before this commit: robot conveyor_belt_dof1, 5 links, 4 joints
Joints:
- joint whisker_left_joint: axis (none) -> 0 1 0
- joint whisker_right_joint: axis (none) -> 0 1 0

Commit message: Finished End Effector. Should test out end effector movements

File: manipulation/models/yaskawa_end_effector_description/urdf/end_effector_3.urdf (robot description, URDF)
Before this commit: robot conveyor_belt_dof1, 5 links, 4 joints
Links:
- link puller_link: mass None -> 0.01
- link pusher_link: mass None -> 0.01
Joints:
- joint whisker_left_joint: axis 0 1 0 -> 1 0 0
- joint whisker_right_joint: axis 0 1 0 -> 1 0 0

Commit message: fixing conveyor belt when its moving fast. It tends to curl itself up.

File: manipulation/models/yaskawa_end_effector_description/urdf/end_effector_3.urdf (robot description, URDF)
Before this commit: robot conveyor_belt_dof1, 5 links, 4 joints
Links:
- link puller_link: geometry collision box size=0.95 0.5 0.01; visual box size=0.95 0.5 0.01

Commit message: fixing pusher and puller confusion. One's moving the other

File: manipulation/models/yaskawa_end_effector_description/urdf/end_effector_3.urdf (robot description, URDF)
Before this commit: robot conveyor_belt_dof1, 5 links, 4 joints
Links:
- link puller_link: mass 0.01 -> 1
- link pusher_link: mass 0.01 -> 1

Commit message: Robot arm now able to take in package and release it to the cabinet. Will need to make small adjustments such as the trajectory points.

File: manipulation/models/yaskawa_end_effector_description/urdf/end_effector_3.urdf (robot description, URDF)
Before this commit: robot conveyor_belt_dof1, 5 links, 4 joints
Links:
- link ee_base: geometry visual mesh filename=../mesh/cbee_gripper_1st-collision.obj
- link puller_link: geometry collision box size=0.95 0.4 0.01
- link pusher_link: geometry collision box size=0.1 0.5 0.25

Commit message: Addd whisker movements. Need to fix whisker movements, increase the puller's gains

File: manipulation/models/yaskawa_end_effector_description/urdf/end_effector_3.urdf (robot description, URDF)
Before this commit: robot conveyor_belt_dof1, 5 links, 4 joints
Links:
- added link left_whisker_offset; visual box size=0.1 0.1 0.1
- added link right_whisker_offset; visual box size=0.1 0.1 0.1
- link puller_link: geometry collision box size=0.95 0.4 0.01; visual box size=0.95 0.4 0.01
- link pusher_link: geometry collision box size=0.1 0.5 0.25; visual box size=0.01 0.5 0.25
- link whisker_left_link: geometry collision box size=0.08 0.39 0.003; collision box size=0.08 0.39 0.003
- link whisker_right_link: geometry collision box size=0.08 0.39 0.003; collision box size=0.08 0.39 0.003
Joints:
- added joint whisker_left_to_base: type fixed, parent ee_base, child left_whisker_offset, origin xyz=0 0.2 0 rpy=0 0 0
- added joint whisker_right_to_base: type fixed, parent ee_base, child right_whisker_offset, origin xyz=0 -0.2 0 rpy=0 0 0
