Commit message: pushing

File: manipulation/models/yaskawa_end_effector_description/urdf/end_effector_4.urdf (robot description, URDF)
Before this commit: robot conveyor_belt_dof1, 7 links, 6 joints
Links:
- removed link puller_link
- removed link pusher_link
- added link roller_link_1, mass 0.01; collision cylinder length=0.5 radius=0.025; visual cylinder length=0.5 radius=0.025
- added link roller_link_2, mass 0.01; collision cylinder length=0.5 radius=0.025; visual cylinder length=0.5 radius=0.025
- added link roller_link_3, mass 0.01; collision cylinder length=0.5 radius=0.025; visual cylinder length=0.5 radius=0.025
- added link roller_link_4, mass 0.01; collision cylinder length=0.5 radius=0.025; visual cylinder length=0.5 radius=0.025
- link ee_base: geometry 
Joints:
- removed joint puller_joint
- removed joint pusher_joint
- added joint roller_joint_1: type revolute, parent ee_base, child roller_link_1, origin xyz=0 0 0 rpy=0 0 0
- added joint roller_joint_2: type revolute, parent ee_base, child roller_link_2, origin xyz=0 0 0 rpy=0 0 0
- added joint roller_joint_3: type revolute, parent ee_base, child roller_link_3, origin xyz=0 0 0 rpy=0 0 0
- added joint roller_joint_4: type revolute, parent ee_base, child roller_link_4, origin xyz=0 0 0 rpy=0 0 0

Commit message: working on end effector. Rollers cannot move with command

File: manipulation/models/yaskawa_end_effector_description/urdf/end_effector_4.urdf (robot description, URDF)
Before this commit: robot conveyor_belt_dof1, 9 links, 8 joints
Links:
- added link roller_base_1; visual box size=0.05 0.05 0.05
- added link roller_base_2; visual box size=0.05 0.05 0.05
- added link roller_base_3; visual box size=0.05 0.05 0.05
- added link roller_base_4; visual box size=0.05 0.05 0.05
- added link roller_base_5; visual box size=0.05 0.05 0.05
- added link roller_link_5, mass 0.01; collision cylinder length=0.5 radius=0.025; visual cylinder length=0.5 radius=0.025
- link roller_link_4: geometry collision cylinder length=0.5 radius=0.02; visual box size=0.04 0.04 0.5
- link whisker_left_link: mass 0.1 -> 0.01
- link whisker_right_link: mass 0.1 -> 0.01
Joints:
- added joint ee_base_to_roller_base_1: type fixed, parent ee_base, child roller_base_1, origin xyz=0.2 0 -0.175 rpy=0 0 0
- added joint ee_base_to_roller_base_2: type fixed, parent ee_base, child roller_base_2, origin xyz=0.3 0 -0.175 rpy=0 0 0
- added joint ee_base_to_roller_base_3: type fixed, parent ee_base, child roller_base_3, origin xyz=0.4 0 -0.175 rpy=0 0 0
- added joint ee_base_to_roller_base_4: type fixed, parent ee_base, child roller_base_4, origin xyz=0.45 0 -0.175 rpy=0 0 0
- added joint ee_base_to_roller_base_5: type fixed, parent ee_base, child roller_base_5, origin xyz=0.5 0 -0.175 rpy=0 0 0
- added joint roller_joint_5: type revolute, parent roller_base_5, child roller_link_5, origin xyz=0 0 0 rpy=0 0 0, axis 0 1 0
- joint roller_joint_1: axis (none) -> 0 1 0; parent ee_base -> roller_base_1
- joint roller_joint_2: axis (none) -> 0 1 0; parent ee_base -> roller_base_2
- joint roller_joint_3: axis (none) -> 0 1 0; parent ee_base -> roller_base_3
- joint roller_joint_4: axis (none) -> 0 1 0; parent ee_base -> roller_base_4

Commit message: in the middle of increasing ee rollers

File: manipulation/models/yaskawa_end_effector_description/urdf/end_effector_4.urdf (robot description, URDF)
Before this commit: robot conveyor_belt_dof1, 15 links, 14 joints
Links:
- added link roller_base_6; visual box size=0.05 0.05 0.05
- added link roller_base_7; visual box size=0.05 0.05 0.05
- added link roller_link_6, mass 0.01; collision cylinder length=0.5 radius=0.02; visual cylinder length=0.5 radius=0.02
- added link roller_link_7, mass 0.01; collision cylinder length=0.5 radius=0.02; visual cylinder length=0.5 radius=0.02
- link roller_link_1: geometry collision cylinder length=0.5 radius=0.02; visual cylinder length=0.5 radius=0.02
- link roller_link_2: geometry collision cylinder length=0.5 radius=0.02; visual cylinder length=0.5 radius=0.02
- link roller_link_3: geometry collision cylinder length=0.5 radius=0.02; visual cylinder length=0.5 radius=0.02
- link roller_link_4: geometry collision cylinder length=0.5 radius=0.02; visual cylinder length=0.5 radius=0.02
- link roller_link_5: geometry collision cylinder length=0.5 radius=0.02; visual cylinder length=0.5 radius=0.02
Joints:
- added joint ee_base_to_roller_base_6: type fixed, parent ee_base, child roller_base_6, origin xyz=0.45 0 -0.175 rpy=0 0 0
- added joint ee_base_to_roller_base_7: type fixed, parent ee_base, child roller_base_7, origin xyz=0.5 0 -0.175 rpy=0 0 0
- added joint roller_joint_6: type revolute, parent roller_base_6, child roller_link_6, origin xyz=0 0 0 rpy=0 0 0, axis 0 1 0
- added joint roller_joint_7: type revolute, parent roller_base_7, child roller_link_7, origin xyz=0 0 0 rpy=0 0 0, axis 0 1 0
- joint ee_base_to_roller_base_2: origin xyz=0.3 0 -0.175 rpy=0 0 0 -> xyz=0.25 0 -0.175 rpy=0 0 0
- joint ee_base_to_roller_base_3: origin xyz=0.4 0 -0.175 rpy=0 0 0 -> xyz=0.3 0 -0.175 rpy=0 0 0
- joint ee_base_to_roller_base_4: origin xyz=0.45 0 -0.175 rpy=0 0 0 -> xyz=0.35 0 -0.175 rpy=0 0 0
- joint ee_base_to_roller_base_5: origin xyz=0.5 0 -0.175 rpy=0 0 0 -> xyz=0.4 0 -0.175 rpy=0 0 0

Commit message: fixed roller issue. New end effector belt is finished. Working to fix issues on whiskers. State seen in primitive_executor is not correct.

File: manipulation/models/yaskawa_end_effector_description/urdf/end_effector_4.urdf (robot description, URDF)
Before this commit: robot conveyor_belt_dof1, 19 links, 18 joints
Links:
- link left_whisker_offset: geometry visual box size=0.01 0.01 0.01
- link right_whisker_offset: geometry visual box size=0.01 0.01 0.01
- link roller_base_1: geometry 
- link roller_base_2: geometry 
- link roller_base_3: geometry 
- link roller_base_4: geometry 
- link roller_base_5: geometry 
- link roller_base_6: geometry 
- link roller_base_7: geometry 
- link roller_link_1: mass 0.01 -> 0.001; geometry collision cylinder length=0.5 radius=0.0225; visual cylinder length=0.5 radius=0.0225
- link roller_link_2: mass 0.01 -> 0.001; geometry collision cylinder length=0.5 radius=0.0225; visual cylinder length=0.5 radius=0.0225
- link roller_link_3: mass 0.01 -> 0.001; geometry collision cylinder length=0.5 radius=0.0225; visual cylinder length=0.5 radius=0.0225
- link roller_link_4: mass 0.01 -> 0.001; geometry collision cylinder length=0.5 radius=0.0225; visual box size=0.04 0.04 0.5
- link roller_link_5: mass 0.01 -> 0.001; geometry collision cylinder length=0.5 radius=0.0225; visual cylinder length=0.5 radius=0.0225
- link roller_link_6: mass 0.01 -> 0.001; geometry collision cylinder length=0.5 radius=0.0225; visual cylinder length=0.5 radius=0.0225
- link roller_link_7: mass 0.01 -> 0.001; geometry collision cylinder length=0.5 radius=0.0225; visual cylinder length=0.5 radius=0.0225
Joints:
- joint ee_base_to_roller_base_1: origin xyz=0.2 0 -0.175 rpy=0 0 0 -> xyz=0.1 0 -0.175 rpy=0 0 0
- joint ee_base_to_roller_base_2: origin xyz=0.25 0 -0.175 rpy=0 0 0 -> xyz=0.15 0 -0.175 rpy=0 0 0
- joint ee_base_to_roller_base_3: origin xyz=0.3 0 -0.175 rpy=0 0 0 -> xyz=0.2 0 -0.175 rpy=0 0 0
- joint ee_base_to_roller_base_4: origin xyz=0.35 0 -0.175 rpy=0 0 0 -> xyz=0.25 0 -0.175 rpy=0 0 0
- joint ee_base_to_roller_base_5: origin xyz=0.4 0 -0.175 rpy=0 0 0 -> xyz=0.3 0 -0.175 rpy=0 0 0
- joint ee_base_to_roller_base_6: origin xyz=0.45 0 -0.175 rpy=0 0 0 -> xyz=0.35 0 -0.175 rpy=0 0 0
- joint ee_base_to_roller_base_7: origin xyz=0.5 0 -0.175 rpy=0 0 0 -> xyz=0.4 0 -0.175 rpy=0 0 0
- joint whisker_left_joint: origin xyz=0.35 0 0 rpy=0 0 0 -> xyz=0 0 0 rpy=0 0 0; parent ee_base -> left_whisker_offset
- joint whisker_left_to_base: origin xyz=0 0.2 0 rpy=0 0 0 -> xyz=0.2 0.275 -0.1 rpy=0 0 0
- joint whisker_right_joint: origin xyz=0.35 0 0 rpy=0 0 0 -> xyz=0 0 0 rpy=0 0 0; parent ee_base -> right_whisker_offset
- joint whisker_right_to_base: origin xyz=0 -0.2 0 rpy=0 0 0 -> xyz=0.2 -0.275 -0.1 rpy=0 0 0

Commit message: commiting

File: manipulation/models/yaskawa_end_effector_description/urdf/end_effector_4.urdf (robot description, URDF)
Before this commit: robot conveyor_belt_dof1, 19 links, 18 joints
Links:
- added link cover_back, mass 0.001; collision box size=0.01 0.35 0.05; visual box size=0.01 0.35 0.05
- added link cover_left, mass 0.001; collision box size=0.01 0.35 0.05; visual box size=0.01 0.35 0.05
- added link cover_right, mass 0.001; collision box size=0.01 0.35 0.05; visual box size=0.01 0.35 0.05
- link ee_base: geometry visual box size=0.01 0.01 0.01
- link roller_link_1: geometry collision cylinder length=0.43 radius=0.0175; visual cylinder length=0.43 radius=0.0175
- link roller_link_2: geometry collision cylinder length=0.43 radius=0.0175; visual cylinder length=0.43 radius=0.0175
- link roller_link_3: geometry collision cylinder length=0.43 radius=0.0175; visual cylinder length=0.43 radius=0.0175
- link roller_link_4: geometry collision cylinder length=0.43 radius=0.0175; visual box size=0.035 0.035 0.43
- link roller_link_5: geometry collision cylinder length=0.43 radius=0.0175; visual cylinder length=0.43 radius=0.0175
- link roller_link_6: geometry collision cylinder length=0.43 radius=0.0175; visual cylinder length=0.43 radius=0.0175
- link roller_link_7: geometry collision cylinder length=0.43 radius=0.0175; visual cylinder length=0.43 radius=0.0175
Joints:
- added joint cover_back_to_base: type fixed, parent ee_base, child cover_back, origin xyz=0.075 0 -0.125 rpy=0 0 0
- added joint cover_left_to_base: type fixed, parent ee_base, child cover_left, origin xyz=0.25 0.2 -0.125 rpy=0 0 1.57
- added joint cover_right_to_base: type fixed, parent ee_base, child cover_right, origin xyz=0.25 -0.2 -0.125 rpy=0 0 1.57
- joint ee_base_to_roller_base_1: origin xyz=0.1 0 -0.175 rpy=0 0 0 -> xyz=0.1 0 -0.175 rpy=1.57 0 0
- joint ee_base_to_roller_base_2: origin xyz=0.15 0 -0.175 rpy=0 0 0 -> xyz=0.15 0 -0.175 rpy=1.57 0 0
- joint ee_base_to_roller_base_3: origin xyz=0.2 0 -0.175 rpy=0 0 0 -> xyz=0.2 0 -0.175 rpy=1.57 0 0
- joint ee_base_to_roller_base_4: origin xyz=0.25 0 -0.175 rpy=0 0 0 -> xyz=0.25 0 -0.175 rpy=1.57 0 0
- joint ee_base_to_roller_base_5: origin xyz=0.3 0 -0.175 rpy=0 0 0 -> xyz=0.3 0 -0.175 rpy=1.57 0 0
- joint ee_base_to_roller_base_6: origin xyz=0.35 0 -0.175 rpy=0 0 0 -> xyz=0.35 0 -0.175 rpy=1.57 0 0
- joint ee_base_to_roller_base_7: origin xyz=0.4 0 -0.175 rpy=0 0 0 -> xyz=0.4 0 -0.175 rpy=1.57 0 0
- joint roller_joint_1: axis 0 1 0 -> 1 0 0
- joint roller_joint_2: axis 0 1 0 -> 1 0 0
- joint roller_joint_3: axis 0 1 0 -> 1 0 0
- joint roller_joint_4: axis 0 1 0 -> 1 0 0
- joint roller_joint_5: axis 0 1 0 -> 1 0 0
- joint roller_joint_6: axis 0 1 0 -> 1 0 0
- joint roller_joint_7: axis 0 1 0 -> 1 0 0

Commit message: finished updating new ee

File: manipulation/models/yaskawa_end_effector_description/urdf/end_effector_4.urdf (robot description, URDF)
Before this commit: robot conveyor_belt_dof1, 22 links, 21 joints
Links:
- added link roller_base_10
- added link roller_base_11
- added link roller_base_8
- added link roller_base_9
- added link roller_link_10, mass 0.001; collision cylinder length=0.43 radius=0.0175; visual cylinder length=0.43 radius=0.0175
- added link roller_link_11, mass 0.001; collision cylinder length=0.43 radius=0.0175; visual cylinder length=0.43 radius=0.0175
- added link roller_link_8, mass 0.001; collision cylinder length=0.43 radius=0.0175; visual cylinder length=0.43 radius=0.0175
- added link roller_link_9, mass 0.001; collision cylinder length=0.43 radius=0.0175; visual cylinder length=0.43 radius=0.0175
- link cover_back: geometry collision box size=0.01 0.43 0.035; visual box size=0.01 0.43 0.035
- link cover_left: geometry collision box size=0.01 0.54 0.035; visual box size=0.01 0.54 0.035
- link cover_right: geometry collision box size=0.01 0.54 0.035; visual box size=0.01 0.54 0.035
- link whisker_right_link: geometry collision box size=0.08 0.37 0.003; collision box size=0.08 0.37 0.003
Joints:
- added joint ee_base_to_roller_base_10: type fixed, parent ee_base, child roller_base_10, origin xyz=0.59875 0 -0.0725 rpy=-1.57 0 0
- added joint ee_base_to_roller_base_11: type fixed, parent ee_base, child roller_base_11, origin xyz=0.65 0 -0.0725 rpy=-1.57 0 0
- added joint ee_base_to_roller_base_8: type fixed, parent ee_base, child roller_base_8, origin xyz=0.49625 0 -0.0725 rpy=-1.57 0 0
- added joint ee_base_to_roller_base_9: type fixed, parent ee_base, child roller_base_9, origin xyz=0.5475 0 -0.0725 rpy=-1.57 0 0
- added joint roller_joint_10: type revolute, parent roller_base_10, child roller_link_10, origin xyz=0 0 0 rpy=0 0 0, axis 0 0 1
- added joint roller_joint_11: type revolute, parent roller_base_11, child roller_link_11, origin xyz=0 0 0 rpy=0 0 0, axis 0 0 1
- added joint roller_joint_8: type revolute, parent roller_base_8, child roller_link_8, origin xyz=0 0 0 rpy=0 0 0, axis 0 0 1
- added joint roller_joint_9: type revolute, parent roller_base_9, child roller_link_9, origin xyz=0 0 0 rpy=0 0 0, axis 0 0 1
- joint cover_back_to_base: origin xyz=0.075 0 -0.125 rpy=0 0 0 -> xyz=0.12 0 -0.0375 rpy=0 0 0
- joint cover_left_to_base: origin xyz=0.25 0.2 -0.125 rpy=0 0 1.57 -> xyz=0.4 0.2225 -0.0375 rpy=0 0 1.57
- joint cover_right_to_base: origin xyz=0.25 -0.2 -0.125 rpy=0 0 1.57 -> xyz=0.4 -0.2225 -0.0375 rpy=0 0 1.57
- joint ee_base_to_roller_base_1: origin xyz=0.1 0 -0.175 rpy=1.57 0 0 -> xyz=0.1375 0 -0.0725 rpy=-1.57 0 0
- joint ee_base_to_roller_base_2: origin xyz=0.15 0 -0.175 rpy=1.57 0 0 -> xyz=0.18875 0 -0.0725 rpy=-1.57 0 0
- joint ee_base_to_roller_base_3: origin xyz=0.2 0 -0.175 rpy=1.57 0 0 -> xyz=0.24 0 -0.0725 rpy=-1.57 0 0
- joint ee_base_to_roller_base_4: origin xyz=0.25 0 -0.175 rpy=1.57 0 0 -> xyz=0.29125 0 -0.0725 rpy=-1.57 0 0
- joint ee_base_to_roller_base_5: origin xyz=0.3 0 -0.175 rpy=1.57 0 0 -> xyz=0.3425 0 -0.0725 rpy=-1.57 0 0
- joint ee_base_to_roller_base_6: origin xyz=0.35 0 -0.175 rpy=1.57 0 0 -> xyz=0.39375 0 -0.0725 rpy=-1.57 0 0
- joint ee_base_to_roller_base_7: origin xyz=0.4 0 -0.175 rpy=1.57 0 0 -> xyz=0.445 0 -0.0725 rpy=-1.57 0 0
- joint roller_joint_1: axis 1 0 0 -> 0 0 1
- joint roller_joint_2: axis 1 0 0 -> 0 0 1
- joint roller_joint_3: axis 1 0 0 -> 0 0 1
- joint roller_joint_4: axis 1 0 0 -> 0 0 1
- joint roller_joint_5: axis 1 0 0 -> 0 0 1
- joint roller_joint_6: axis 1 0 0 -> 0 0 1
- joint roller_joint_7: axis 1 0 0 -> 0 0 1
- joint whisker_left_to_base: origin xyz=0.2 0.275 -0.1 rpy=0 0 0 -> xyz=0.385 0.255 -0.02 rpy=0 0 0
- joint whisker_right_to_base: origin xyz=0.2 -0.275 -0.1 rpy=0 0 0 -> xyz=0.385 -0.255 -0.02 rpy=0 0 0

Commit message: finished for now

File: manipulation/models/yaskawa_end_effector_description/urdf/end_effector_4.urdf (robot description, URDF)
Before this commit: robot conveyor_belt_dof1, 30 links, 29 joints
Links:
- link whisker_left_link: geometry collision box size=0.08 0.37 0.003; collision box size=0.08 0.37 0.003
- link whisker_right_link: geometry collision box size=0.08 0.37 0.003; collision box size=0.08 0.37 0.003
